File: keyboard-tutorial.kicad_sch (KiCad schematic)
At the start: 24 parts, among them SW1 SW_Push, U1 ATmega32U4-A, Y1 16MHz

Commit message: update
Parts:
- MX1, MX2, MX3, MX4: footprint MX_Alps_Hybrid:MX-10U-NoLED -> MX_Alps_Hybrid:MX-1U-NoLED
Changed lines of the file:
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@@
       (effects (font (size 0.508 0.508)))
     )
-    (property "Footprint" "MX_Alps_Hybrid:MX-10U-NoLED" (id 2) (at 198.755 116.205 0)
+    (property "Footprint" "MX_Alps_Hybrid:MX-1U-NoLED" (id 2) (at 198.755 116.205 0)
       (effects (font (size 1.524 1.524)) hide)
     )
@@
       (effects (font (size 0.508 0.508)))
     )
-    (property "Footprint" "MX_Alps_Hybrid:MX-10U-NoLED" (id 2) (at 183.515 132.715 0)
+    (property "Footprint" "MX_Alps_Hybrid:MX-1U-NoLED" (id 2) (at 183.515 132.715 0)
       (effects (font (size 1.524 1.524)) hide)
     )
@@
       (effects (font (size 0.508 0.508)))
     )
-    (property "Footprint" "MX_Alps_Hybrid:MX-10U-NoLED" (id 2) (at 198.755 132.715 0)
+    (property "Footprint" "MX_Alps_Hybrid:MX-1U-NoLED" (id 2) (at 198.755 132.715 0)
       (effects (font (size 1.524 1.524)) hide)
     )
@@
       (effects (font (size 0.508 0.508)))
     )
-    (property "Footprint" "MX_Alps_Hybrid:MX-10U-NoLED" (id 2) (at 183.515 116.205 0)
+    (property "Footprint" "MX_Alps_Hybrid:MX-1U-NoLED" (id 2) (at 183.515 116.205 0)
       (effects (font (size 1.524 1.524)) hide)
     )
@@
     )
     (path "/f1cf35b0-3c50-4cb3-8138-22c3a5a5c0d3"
-      (reference "MX1") (unit 1) (value "MX-NoLED") (footprint "MX_Alps_Hybrid:MX-10U-NoLED")
+      (reference "MX1") (unit 1) (value "MX-NoLED") (footprint "MX_Alps_Hybrid:MX-1U-NoLED")
     )
     (path "/9bc6cbf6-b847-46a4-a12c-65fd97eb6dcf"
-      (reference "MX2") (unit 1) (value "MX-NoLED") (footprint "MX_Alps_Hybrid:MX-10U-NoLED")
+      (reference "MX2") (unit 1) (value "MX-NoLED") (footprint "MX_Alps_Hybrid:MX-1U-NoLED")
     )
     (path "/13b76eee-4ee3-40c9-bef8-281e49bc9de6"
-      (reference "MX3") (unit 1) (value "MX-NoLED") (footprint "MX_Alps_Hybrid:MX-10U-NoLED")
+      (reference "MX3") (unit 1) (value "MX-NoLED") (footprint "MX_Alps_Hybrid:MX-1U-NoLED")
     )
     (path "/ef142a89-d1f5-4726-8e35-af9d3862c1f7"
-      (reference "MX4") (unit 1) (value "MX-NoLED") (footprint "MX_Alps_Hybrid:MX-10U-NoLED")
+      (reference "MX4") (unit 1) (value "MX-NoLED") (footprint "MX_Alps_Hybrid:MX-1U-NoLED")
     )
     (path "/1f71df7b-636a-4718-aabe-f0920f9ed737"

Commit message: Keyboard settings updates
Connections:
- net D+: now also USB1.3 (D+); no longer USB1.4 (D-)
- net D-: now also USB1.4 (D-); no longer USB1.5 (VBUS)
- net VCC: now also USB1.5 (VBUS); no longer USB1.6 (SHIELD)
Other:
- moved on the sheet: F1
Changed lines of the file:
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@@
   (junction (at 93.98 50.8) (diameter 0) (color 0 0 0 0)
   )
+  (junction (at 196.85 67.31) (diameter 0) (color 0 0 0 0)
+  )
   (junction (at 53.34 60.96) (diameter 0) (color 0 0 0 0)
   )
@@
   (junction (at 73.66 110.49) (diameter 0) (color 0 0 0 0)
   )
-  (junction (at 195.58 64.77) (diameter 0) (color 0 0 0 0)
-  )
   (junction (at 60.96 110.49) (diameter 0) (color 0 0 0 0)
   )
@@
     (stroke (width 0) (type default) (color 0 0 0 0))
   )
-  (wire (pts (xy 189.23 77.47) (xy 191.77 77.47))
+  (wire (pts (xy 189.23 77.47) (xy 190.5 77.47))
     (stroke (width 0) (type default) (color 0 0 0 0))
   )
@@
     (stroke (width 0) (type default) (color 0 0 0 0))
   )
+  (wire (pts (xy 189.23 67.31) (xy 196.85 67.31))
+    (stroke (width 0) (type default) (color 0 0 0 0))
+  )
   (wire (pts (xy 186.69 140.97) (xy 194.31 140.97))
     (stroke (width 0) (type default) (color 0 0 0 0))
@@
     (stroke (width 0) (type default) (color 0 0 0 0))
   )
-  (wire (pts (xy 208.28 64.77) (xy 219.71 64.77))
+  (wire (pts (xy 209.55 67.31) (xy 217.17 67.31))
     (stroke (width 0) (type default) (color 0 0 0 0))
   )
@@
     (stroke (width 0) (type default) (color 0 0 0 0))
   )
-  (wire (pts (xy 189.23 64.77) (xy 195.58 64.77))
-    (stroke (width 0) (type default) (color 0 0 0 0))
-  )
   (wire (pts (xy 93.98 36.83) (xy 93.98 38.1))
     (stroke (width 0) (type default) (color 0 0 0 0))
@@
     (stroke (width 0) (type default) (color 0 0 0 0))
   )
-  (wire (pts (xy 195.58 64.77) (xy 203.2 64.77))
+  (wire (pts (xy 196.85 67.31) (xy 204.47 67.31))
     (stroke (width 0) (type default) (color 0 0 0 0))
   )
@@
     )
   )
-  (global_label "D+" (shape input) (at 189.23 69.85 0) (fields_autoplaced)
+  (global_label "D+" (shape input) (at 189.23 72.39 0) (fields_autoplaced)
     (effects (font (size 1.2 1.2)) (justify left))
-    (property "Intersheet References" "${INTERSHEET_REFS}" (id 0) (at 194.1957 69.775 0)
+    (property "Intersheet References" "${INTERSHEET_REFS}" (id 0) (at 194.1957 72.315 0)
       (effects (font (size 1.2 1.2)) (justify left) hide)
     )
@@
     )
   )
-  (global_label "D-" (shape input) (at 189.23 67.31 0) (fields_autoplaced)
+  (global_label "D-" (shape input) (at 189.23 69.85 0) (fields_autoplaced)
     (effects (font (size 1.2 1.2)) (justify left))
-    (property "Intersheet References" "${INTERSHEET_REFS}" (id 0) (at 194.1957 67.235 0)
+    (property "Intersheet References" "${INTERSHEET_REFS}" (id 0) (at 194.1957 69.775 0)
       (effects (font (size 1.2 1.2)) (justify left) hide)
     )
@@
     (pin "2")
   )
-  (symbol (lib_id "power:GND") (at 191.77 77.47 0) (unit 1)
-    (in_bom yes) (on_board yes) (fields_autoplaced)
-    (property "Reference" "#PWR0112" (id 0) (at 191.77 83.82 0)
-      (effects (font (size 1.27 1.27)) hide)
-    )
-    (property "Value" "GND" (id 1) (at 191.77 82.55 0))
-    (property "Footprint" "" (id 2) (at 191.77 77.47 0)
-      (effects (font (size 1.27 1.27)) hide)
-    )
-    (property "Datasheet" "" (id 3) (at 191.77 77.47 0)
+  (symbol (lib_id "power:GND") (at 190.5 77.47 0) (unit 1)
+    (in_bom yes) (on_board yes) (fields_autoplaced)
+    (property "Reference" "#PWR0112" (id 0) (at 190.5 83.82 0)
+      (effects (font (size 1.27 1.27)) hide)
+    )
+    (property "Value" "GND" (id 1) (at 190.5 82.55 0))
+    (property "Footprint" "" (id 2) (at 190.5 77.47 0)
+      (effects (font (size 1.27 1.27)) hide)
+    )
+    (property "Datasheet" "" (id 3) (at 190.5 77.47 0)
       (effects (font (size 1.27 1.27)) hide)
     )
@@
     (pin "1")
   )
-  (symbol (lib_id "power:+5V") (at 219.71 64.77 0) (unit 1)
-    (in_bom yes) (on_board yes) (fields_autoplaced)
-    (property "Reference" "#PWR0113" (id 0) (at 219.71 68.58 0)
-      (effects (font (size 1.27 1.27)) hide)
-    )
-    (property "Value" "+5V" (id 1) (at 219.71 59.69 0))
-    (property "Footprint" "" (id 2) (at 219.71 64.77 0)
-      (effects (font (size 1.27 1.27)) hide)
-    )
-    (property "Datasheet" "" (id 3) (at 219.71 64.77 0)
-      (effects (font (size 1.27 1.27)) hide)
-    )
-    (pin "1")
-  )
-  (symbol (lib_id "Device:Polyfuse_Small") (at 205.74 64.77 90) (unit 1)
-    (in_bom yes) (on_board yes) (fields_autoplaced)
-    (property "Reference" "F1" (id 0) (at 205.74 58.42 90))
-    (property "Value" "500mA" (id 1) (at 205.74 60.96 90))
-    (property "Footprint" "Fuse:Fuse_1206_3216Metric" (id 2) (at 210.82 63.5 0)
+  (symbol (lib_id "power:+5V") (at 217.17 67.31 0) (unit 1)
+    (in_bom yes) (on_board yes) (fields_autoplaced)
+    (property "Reference" "#PWR0113" (id 0) (at 217.17 71.12 0)
+      (effects (font (size 1.27 1.27)) hide)
+    )
+    (property "Value" "+5V" (id 1) (at 217.17 62.23 0))
+    (property "Footprint" "" (id 2) (at 217.17 67.31 0)
+      (effects (font (size 1.27 1.27)) hide)
+    )
+    (property "Datasheet" "" (id 3) (at 217.17 67.31 0)
+      (effects (font (size 1.27 1.27)) hide)
+    )
+    (pin "1")
+  )
+  (symbol (lib_id "Device:Polyfuse_Small") (at 207.01 67.31 90) (unit 1)
+    (in_bom yes) (on_board yes) (fields_autoplaced)
+    (property "Reference" "F1" (id 0) (at 207.01 60.96 90))
+    (property "Value" "500mA" (id 1) (at 207.01 63.5 90))
+    (property "Footprint" "Fuse:Fuse_1206_3216Metric" (id 2) (at 212.09 66.04 0)
       (effects (font (size 1.27 1.27)) (justify left) hide)
     )
-    (property "Datasheet" "~" (id 3) (at 205.74 64.77 0)
+    (property "Datasheet" "~" (id 3) (at 207.01 67.31 0)
       (effects (font (size 1.27 1.27)) hide)
     )
@@
     (pin "2")
   )
-  (symbol (lib_id "power:VCC") (at 195.58 64.77 0) (unit 1)
-    (in_bom yes) (on_board yes) (fields_autoplaced)
-    (property "Reference" "#PWR0111" (id 0) (at 195.58 68.58 0)
-      (effects (font (size 1.27 1.27)) hide)
-    )
-    (property "Value" "VCC" (id 1) (at 195.58 59.69 0))
-    (property "Footprint" "" (id 2) (at 195.58 64.77 0)
-      (effects (font (size 1.27 1.27)) hide)
-    )
-    (property "Datasheet" "" (id 3) (at 195.58 64.77 0)
-      (effects (font (size 1.27 1.27)) hide)
-    )
+  (symbol (lib_id "power:VCC") (at 196.85 67.31 0) (unit 1)
+    (in_bom yes) (on_board yes) (fields_autoplaced)
+    (property "Reference" "#PWR0111" (id 0) (at 196.85 71.12 0)
+      (effects (font (size 1.27 1.27)) hide)
+    )
+    (property "Value" "VCC" (id 1) (at 196.85 62.23 0))
+    (property "Footprint" "" (id 2) (at 196.85 67.31 0)
+      (effects (font (size 1.27 1.27)) hide)
+    )
+    (property "Datasheet" "" (id 3) (at 196.85 67.31 0)
+      (effects (font (size 1.27 1.27)) hide)
+    )
